File: hardware/EDA-Files/UP1-Progger/UP1-Progger.kicad_sch (KiCad schematic)
At the start: 12 parts, among them J1 UP1_Prog_Connector, J11 UP1_Prog_Connector, J2 USB_B_Micro, J3 Conn_01x03, J4 SWD_Interface, J5 ST Link V2 Clone, SW1 Reset, SW2 Bootsel, U1 LDO_3V3_SOT23-3

Commit message: UP1-Progger V02.00
Parts:
- removed J1: UP1_Prog_Connector, Connector_PinSocket_1.27mm:PinSocket_1x08_P1.27mm_Vertical, symbol OpenKNX:OpenKNX_UP1_Prog_Connector
- removed J2: USB_B_Micro, DomsKiCADLib:USB_Micro-B_JING_C10418, symbol REG1-Controller2040-rescue:USB_B_Micro-Connector
- removed J3: Conn_01x03, Connector_PinHeader_2.54mm:PinHeader_1x03_P2.54mm_Vertical, symbol Connector_Generic:Conn_01x03
- removed J5: ST Link V2 Clone, Connector_IDC:IDC-Header_2x05_P2.54mm_Vertical, symbol Connector_Generic:Conn_02x05_Odd_Even
- added J1: TYPE-C_16PIN_2MD(073), EasyEDALib:USB-C-SMD_TYPE-C-6PIN-2MD-073, symbol EasyEDALib:TYPE-C_16PIN_2MD(073)
- added J10: UP1_Prog_125, EasyEDALib:CONN-SMD_8P-P1.00_MEGASTAR_ZX-SH1.0-8PWT, symbol OpenKNX:OpenKNX_UP1_Prog_Connector
- added LED1: USB-Power, Diode_SMD:D_0603_1608Metric, symbol Device:LED
- added LED2: Device_Pwr, Diode_SMD:D_0603_1608Metric, symbol Device:LED
- added R1, R2: 2k, Resistor_SMD:R_0402_1005Metric, symbol Device:R
- added R3, R4: 5k1, Resistor_SMD:R_0402_1005Metric, symbol Device:R
- added SW3: SW_SPDT, EasyEDALib:SW-SMD_K3-1280S-K1, symbol Switch:SW_SPDT
- C1, C2: LCSC C15849 -> (none)
- D1: LCSC C191023 -> (none)
- J11: value UP1_Prog_Connector -> UP1_Prog_10; footprint EasyEDALib:CONN-TH_1.25-8A -> EasyEDALib:CONN-SMD_8P-P1.25-L4.4-W14.8; LCSC C17700401 -> (none)
- J4: footprint Connector_PinHeader_1.27mm:PinHeader_2x05_P1.27mm_Vertical -> EasyEDALib:IDC-SMD_10P-P1.27-3220-10-0300-00; JLCPCB Rotation Offset -90 -> (none); LCSC C2935953 -> (none)
- SW1, SW2: LCSC C455282 -> (none)
- U1: LCSC C5446 -> (none)
Connections:
- net +3.3V: now also SW3.2 (B); no longer J11.2 (3V3), J4.1 (Pin_1)
- net +5V: now also J1.11 (VBUS), J1.2 (VBUS)
- net Bootsel: now also J10.8 (Bootsel)
- net D+: now also J1.6 (DP1), J1.8 (DP2), J10.4 (D+)
- net D-: now also J1.5 (DN2), J1.7 (DN1), J10.3 (D-)
- net GND: now also J11.0, J11.10, J11.9, J1.1 (GND), J1.12 (GND), J10.0, J10.1 (GND), J10.10, J10.9, R1.1, R2.1, R3.2, R4.2
- net Reset: now also J10.7 (Run)
- net SWCLK: now also J10.5 (SWCLK)
- net SWDIO: now also J10.6 (SWDIO)
- net at C2.1, D1.2 (A), U1.2 (VO): now also LED1.2 (A)
- new net: J10.2 (3V3), J11.2 (3V3), J4.1 (Pin_1), LED2.2 (A), SW3.3 (C)
- new net: LED1.1 (K), R1.2
- new net: J1.4 (CC1), R3.1
- new net: J1.10 (CC2), R4.1
- new net: LED2.1 (K), R2.2
Other:
- moved on the sheet: J11, J4
