File: hardware/EDA-Files/UP1-PM-HF/UP1-PM-HF.kicad_sch (KiCad schematic)
At the start: 10 parts, among them J100 KNX_Conn, SW100 Prog

Commit message: UP1-PM-HF V00.21 * variable Flash (W25Q) * move FP to OpenKNX KiCAD Lib * increase Pad size for hand solder pins * change RP2040 reset circuit
Parts:
- GN100: footprint OpenKNX:NanoBCU_PinHeader_SMD_low_profile -> OpenKNX:NanoBCU_PinHeader_SMD_low_profile_bigPads
Changed lines of the file:
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@@
 	(title_block
 		(title "UP1-PM-HF")
-		(date "2025-12-09")
-		(rev "V00.20")
+		(date "2026-02-06")
+		(rev "V00.21")
 		(company "OpenKNX")
 		(comment 1 "by Ing-Dom <dom@ing-dom.de>")
@@
 			)
 		)
-		(property "Footprint" "OpenKNX:NanoBCU_PinHeader_SMD_low_profile"
+		(property "Footprint" "OpenKNX:NanoBCU_PinHeader_SMD_low_profile_bigPads"
 			(at 29.21 60.96 0)
 			(effects
